File: frontend/hw/interface/interface.kicad_pcb (KiCad board)
At the start: 2 copper layers, 60.2 x 34.5 mm, 11 parts, among them J1 Conn_01x05, J2 Conn_01x05, J3 Conn_01x06, J4 Conn_01x13, J5 Conn_02x13_Odd_Even

Commit message: Add power connector.
Parts:
- added J6: Conn_01x02, Connector_JST:JST_XH_S2B-XH-A_1x02_P2.50mm_Horizontal, F.Cu at (67.8, 94.3)
Routing:
- net +5V: track 46.5 -> 58.0 mm
- net GND: track 107.9 -> 112.9 mm
Changed lines of the file:
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@@
+    )
+  )
+  (footprint "Connector_JST:JST_XH_S2B-XH-A_1x02_P2.50mm_Horizontal" (layer "F.Cu")
+    (at 67.797 94.341 90)
+    (descr "JST XH series connector, S2B-XH-A (http://www.jst-mfg.com/product/pdf/eng/eXH.pdf), generated with kicad-footprint-generator")
+    (tags "connector JST XH horizontal")
+    (property "Sheetfile" "interface.kicad_sch")
+    (property "Sheetname" "")
+    (attr through_hole)
+    (fp_text reference "J6" (at 1.25 -3.5 90) (layer "F.SilkS")
+      (effects (font (size 1 1) (thickness 0.15)))
+    )
+    (fp_text value "Conn_01x02" (at 1.25 10.4 90) (layer "F.Fab")
+      (effects (font (size 1 1) (thickness 0.15)))
+    )
+    (fp_text user "${REFERENCE}" (at 1.25 3.45 90) (layer "F.Fab")
+      (effects (font (size 1 1) (thickness 0.15)))
+    )
+    (fp_line (start 5.06 9.31) (end 5.06 -2.41) (layer "F.SilkS") (width 0.12))
+    (fp_line (start 3.64 2.09) (end 1.25 2.09) (layer "F.SilkS") (width 0.12))
+    (fp_line (start -0.25 3.2) (end -0.25 8.7) (layer "F.SilkS") (width 0.12))
+    (fp_line (start 2.25 3.2) (end 2.25 8.7) (layer "F.SilkS") (width 0.12))
+    (fp_line (start 0.25 8.7) (end 0.25 3.2) (layer "F.SilkS") (width 0.12))
+    (fp_line (start 1.25 9.31) (end 5.06 9.31) (layer "F.SilkS") (width 0.12))
+    (fp_line (start 2.75 3.2) (end 2.25 3.2) (layer "F.SilkS") (width 0.12))
+    (fp_line (start 5.06 -2.41) (end 3.64 -2.41) (layer "F.SilkS") (width 0.12))
+    (fp_line (start 3.64 -2.41) (end 3.64 2.09) (layer "F.SilkS") (width 0.12))
+    (fp_line (start -1.14 2.09) (end 1.25 2.09) (layer "F.SilkS") (width 0.12))
+    (fp_line (start 0.25 3.2) (end -0.25 3.2) (layer "F.SilkS") (width 0.12))
+    (fp_line (start 0.3 -2.1) (end 0 -1.5) (layer "F.SilkS") (width 0.12))
+    (fp_line (start -2.56 9.31) (end -2.56 -2.41) (layer "F.SilkS") (width 0.12))
+    (fp_line (start 2.25 8.7) (end 2.75 8.7) (layer "F.SilkS") (width 0.12))
+    (fp_line (start -1.14 -2.41) (end -1.14 2.09) (layer "F.SilkS") (width 0.12))
+    (fp_line (start 2.75 8.7) (end 2.75 3.2) (layer "F.SilkS") (width 0.12))
+    (fp_line (start -0.25 8.7) (end 0.25 8.7) (layer "F.SilkS") (width 0.12))
+    (fp_line (start 0 -1.5) (end -0.3 -2.1) (layer "F.SilkS") (width 0.12))
+    (fp_line (start -0.3 -2.1) (end 0.3 -2.1) (layer "F.SilkS") (width 0.12))
+    (fp_line (start -2.56 -2.41) (end -1.14 -2.41) (layer "F.SilkS") (width 0.12))
+    (fp_line (start 1.25 9.31) (end -2.56 9.31) (layer "F.SilkS") (width 0.12))
+    (fp_line (start 5.45 9.7) (end 5.45 -2.8) (layer "F.CrtYd") (width 0.05))
+    (fp_line (start -2.95 9.7) (end 5.45 9.7) (layer "F.CrtYd") (width 0.05))
+    (fp_line (start -2.95 -2.8) (end -2.95 9.7) (layer "F.CrtYd") (width 0.05))
+    (fp_line (start 5.45 -2.8) (end -2.95 -2.8) (layer "F.CrtYd") (width 0.05))
+    (fp_line (start 4.95 9.2) (end 4.95 -2.3) (layer "F.Fab") (width 0.1))
+    (fp_line (start -2.45 9.2) (end -2.45 -2.3) (layer "F.Fab") (width 0.1))
+    (fp_line (start 1.25 9.2) (end -2.45 9.2) (layer "F.Fab") (width 0.1))
+    (fp_line (start -2.45 -2.3) (end -1.25 -2.3) (layer "F.Fab") (width 0.1))
+    (fp_line (start 1.25 9.2) (end 4.95 9.2) (layer "F.Fab") (width 0.1))
+    (fp_line (start 4.95 -2.3) (end 3.75 -2.3) (layer "F.Fab") (width 0.1))
+    (fp_line (start 3.75 2.2) (end 1.25 2.2) (layer "F.Fab") (width 0.1))
+    (fp_line (start 0 1.2) (end 0.625 2.2) (layer "F.Fab") (width 0.1))
+    (fp_line (start -1.25 -2.3) (end -1.25 2.2) (layer "F.Fab") (width 0.1))
+    (fp_line (start -0.625 2.2) (end 0 1.2) (layer "F.Fab") (width 0.1))
+    (fp_line (start -1.25 2.2) (end 1.25 2.2) (layer "F.Fab") (width 0.1))
+    (fp_line (start 3.75 -2.3) (end 3.75 2.2) (layer "F.Fab") (width 0.1))
+    (pad "1" thru_hole roundrect (at 0 0 90) (size 1.7 2) (drill 1) (layers *.Cu *.Mask) (roundrect_rratio 0.147059)
+      (net 1 "+5V") (pinfunction "Pin_1") (pintype "passive"))
+    (pad "2" thru_hole oval (at 2.5 0 90) (size 1.7 2) (drill 1) (layers *.Cu *.Mask)
+      (net 2 "GND") (pinfunction "Pin_2") (pintype "passive"))
+    (model "${KICAD6_3DMODEL_DIR}/Connector_JST.3dshapes/JST_XH_S2B-XH-A_1x02_P2.50mm_Horizontal.wrl"
+      (offset (xyz 0 0 0))
+      (scale (xyz 1 1 1))
+      (rotate (xyz 0 0 0))
     )
   )
@@
   (segment (start 76.764 100.304) (end 75.264489 98.804489) (width 1) (layer "B.Cu") (net 1))
   (segment (start 50 80) (end 51.549511 81.549511) (width 1) (layer "B.Cu") (net 1))
+  (segment (start 70.801 94.341) (end 76.764 100.304) (width 1) (layer "B.Cu") (net 1))
   (segment (start 58.197511 98.804489) (end 56.698 100.304) (width 1) (layer "B.Cu") (net 1))
   (segment (start 51.549511 81.549511) (end 51.549511 82.741806) (width 1) (layer "B.Cu") (net 1))
+  (segment (start 67.797 94.341) (end 70.801 94.341) (width 1) (layer "B.Cu") (net 1))
   (segment (start 54.61 85.802295) (end 54.61 89.916) (width 1) (layer "B.Cu") (net 1))
   (segment (start 62.992 93.218) (end 63.5645 93.7905) (width 1) (layer "F.Cu") (net 2))
+  (segment (start 67.797 91.841) (end 65.4895 91.841) (width 1) (layer "F.Cu") (net 2))
   (segment (start 96.921 80.02) (end 98.281 81.38) (width 1) (layer "F.Cu") (net 2))
+  (segment (start 65.4895 91.841) (end 63.5645 89.916) (width 1) (layer "F.Cu") (net 2))
   (segment (start 93.218 80.02) (end 96.921 80.02) (width 1) (layer "F.Cu") (net 2))
   (segment (start 61.722 93.218) (end 62.992 93.218) (width 1) (layer "F.Cu") (net 2))
