File: frontend/hw/interface/interface.kicad_sch (KiCad schematic)
At the start: 11 parts, among them J1 Conn_01x05, J2 Conn_01x05, J3 Conn_01x06, J4 Conn_01x13, J5 Conn_02x13_Odd_Even

Commit message: Fix 3D view.
Parts:
- J4: footprint Connector_PinHeader_2.54mm:PinHeader_1x13_P2.54mm_Vertical -> Connector_PinSocket_2.54mm:PinSocket_1x13_P2.54mm_Vertical
- J5: footprint Connector_PinHeader_2.54mm:PinHeader_2x13_P2.54mm_Vertical -> Connector_PinSocket_2.54mm:PinSocket_2x13_P2.54mm_Vertical
Changed lines of the file:
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@@
     (property "Reference" "J5" (id 0) (at 165.354 71.4715 0))
     (property "Value" "Conn_02x13_Odd_Even" (id 1) (at 165.354 74.2466 0))
-    (property "Footprint" "Connector_PinHeader_2.54mm:PinHeader_2x13_P2.54mm_Vertical" (id 2) (at 166.624 91.948 0)
+    (property "Footprint" "Connector_PinSocket_2.54mm:PinSocket_2x13_P2.54mm_Vertical" (id 2) (at 166.624 91.948 0)
       (effects (font (size 1.27 1.27)) hide)
     )
@@
       (effects (font (size 1.27 1.27)) (justify left))
     )
-    (property "Footprint" "Connector_PinHeader_2.54mm:PinHeader_1x13_P2.54mm_Vertical" (id 2) (at 79.248 95.25 0)
+    (property "Footprint" "Connector_PinSocket_2.54mm:PinSocket_1x13_P2.54mm_Vertical" (id 2) (at 79.248 95.25 0)
       (effects (font (size 1.27 1.27)) hide)
     )
@@
     )
     (path "/e2d0dbca-b126-4dea-80f2-d802bd17caff"
-      (reference "J4") (unit 1) (value "Conn_01x13") (footprint "Connector_PinHeader_2.54mm:PinHeader_1x13_P2.54mm_Vertical")
+      (reference "J4") (unit 1) (value "Conn_01x13") (footprint "Connector_PinSocket_2.54mm:PinSocket_1x13_P2.54mm_Vertical")
     )
     (path "/c04a157c-b2cc-401d-a361-08484aea24c3"
-      (reference "J5") (unit 1) (value "Conn_02x13_Odd_Even") (footprint "Connector_PinHeader_2.54mm:PinHeader_2x13_P2.54mm_Vertical")
+      (reference "J5") (unit 1) (value "Conn_02x13_Odd_Even") (footprint "Connector_PinSocket_2.54mm:PinSocket_2x13_P2.54mm_Vertical")
     )
     (path "/14202ecb-5941-455d-a867-b86716db90d7"

Commit message: Add power connector.
Parts:
- added J6: Conn_01x02, Connector_JST:JST_XH_S2B-XH-A_1x02_P2.50mm_Horizontal, symbol Connector_Generic:Conn_01x02
Connections:
- net +5V: now also J6.1 (Pin_1)
- net GND: now also J6.2 (Pin_2)
Other:
- moved on the sheet: C1
