File: frontend/pcb/relay/relay.kicad_sch (KiCad schematic)
At the start: 17 parts, among them J1 Conn_01x02, J2 Conn_01x02, J3 CONN_01X02, J4 Conn_01x02, K1 G6B-1114C-US5DC, Q3 BSS138, U2 DSN-MINI-360

Commit message: Finish relay board.
Parts:
- removed H1, H3: MountingHole, MountingHole:MountingHole_3.2mm_M3, symbol Mechanical:MountingHole
- removed J1, J4: Conn_01x02, Connector_JST:JST_XH_B2B-XH-A_1x02_P2.50mm_Vertical, symbol Connector_Generic:Conn_01x02
- added J1: Conn_01x03, Connector_PinSocket_2.54mm:PinSocket_1x03_P2.54mm_Vertical, symbol Connector_Generic:Conn_01x03
- renumbered H4 to H1
Connections:
- net +5V: now also J1.3 (Pin_3)
- net GND: now also J3.1 (Pin_1), J1.1 (Pin_1); no longer J3.2 (Pin_2)
- net Relay: now also J1.2 (Pin_2)
- net at K1.4: now also J3.2 (Pin_2); no longer J3.1 (Pin_1)
Other:
- note added: "To main PCB"
- note removed: "12V out"
- moved on the sheet: C5, D1, D2, H1, J2, J3, K1, Q3, R3, R4, U2

Commit message: Add filter resistor.
Parts:
- added R1: 4R7, Resistor_SMD:R_0603_1608Metric, symbol Device:R
- renumbered C5 to C1, Q3 to Q1, R4 to R2, U2 to U1
Connections:
- net +5V: now also R1.2; no longer C1.1, D2.1 (K), K1.2
- new net: C1.1, D2.1 (K), K1.2, R1.1
Changed lines of the file:
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@@
+    (stroke (width 0) (type default))
+  )
+  (wire (pts (xy 102.87 110.49) (xy 100.33 110.49))
     (stroke (width 0) (type default))
   )
@@
   )
   (wire (pts (xy 55.88 139.7) (xy 41.91 139.7))
+    (stroke (width 0) (type default))
+  )
+  (wire (pts (xy 102.87 107.95) (xy 102.87 110.49))
     (stroke (width 0) (type default))
   )
@@
   (symbol (lib_id "Device:Q_NMOS_GSD") (at 68.58 135.89 0) (mirror y) (unit 1)
     (in_bom yes) (on_board yes) (dnp no)
-    (property "Reference" "Q3" (at 63.373 134.7216 0)
+    (property "Reference" "Q1" (at 63.373 134.7216 0)
       (effects (font (size 1.27 1.27)) (justify left))
     )
@@
       (project "relay"
         (path "/212a0d71-cc7b-49f8-b4ca-a935e5355dca"
-          (reference "Q3") (unit 1)
+          (reference "Q1") (unit 1)
         )
       )
@@
   (symbol (lib_id "dsnmini360:DSN-MINI-360") (at 55.88 54.61 0) (unit 1)
     (in_bom yes) (on_board yes) (dnp no) (fields_autoplaced)
-    (property "Reference" "U2" (at 55.88 46.99 0)
+    (property "Reference" "U1" (at 55.88 46.99 0)
       (effects (font (size 1.27 1.27)))
     )
@@
       (project "relay"
         (path "/212a0d71-cc7b-49f8-b4ca-a935e5355dca"
-          (reference "U2") (unit 1)
+          (reference "U1") (unit 1)
         )
       )
@@
   (symbol (lib_id "Device:R") (at 85.09 135.89 90) (mirror x) (unit 1)
     (in_bom yes) (on_board yes) (dnp no)
-    (property "Reference" "R4" (at 85.09 137.922 90)
+    (property "Reference" "R2" (at 85.09 137.922 90)
       (effects (font (size 1.27 1.27)))
     )
@@
       (project "relay"
         (path "/212a0d71-cc7b-49f8-b4ca-a935e5355dca"
-          (reference "R4") (unit 1)
+          (reference "R2") (unit 1)
         )
       )
@@
     )
   )
-  (symbol (lib_id "power:+5V") (at 92.71 110.49 270) (mirror x) (unit 1)
-    (in_bom yes) (on_board yes) (dnp no)
-    (property "Reference" "#PWR023" (at 88.9 110.49 0)
-      (effects (font (size 1.27 1.27)) hide)
-    )
-    (property "Value" "+5V" (at 96.266 110.49 0)
-      (effects (font (size 1.27 1.27)))
-    )
-    (property "Footprint" "" (at 92.71 110.49 0)
-      (effects (font (size 1.27 1.27)) hide)
-    )
-    (property "Datasheet" "" (at 92.71 110.49 0)
+  (symbol (lib_id "power:+5V") (at 102.87 107.95 0) (mirror y) (unit 1)
+    (in_bom yes) (on_board yes) (dnp no)
+    (property "Reference" "#PWR023" (at 102.87 111.76 0)
+      (effects (font (size 1.27 1.27)) hide)
+    )
+    (property "Value" "+5V" (at 102.87 104.394 0)
+      (effects (font (size 1.27 1.27)))
+    )
+    (property "Footprint" "" (at 102.87 107.95 0)
+      (effects (font (size 1.27 1.27)) hide)
+    )
+    (property "Datasheet" "" (at 102.87 107.95 0)
       (effects (font (size 1.27 1.27)) hide)
     )
@@
     )
   )
+  (symbol (lib_id "Device:R") (at 96.52 110.49 90) (unit 1)
+    (in_bom yes) (on_board yes) (dnp no) (fields_autoplaced)
+    (property "Reference" "R1" (at 96.52 105.41 90)
+      (effects (font (size 1.27 1.27)))
+    )
+    (property "Value" "4R7" (at 96.52 107.95 90)
+      (effects (font (size 1.27 1.27)))
+    )
+    (property "Footprint" "Resistor_SMD:R_0603_1608Metric" (at 96.52 112.268 90)
+      (effects (font (size 1.27 1.27)) hide)
+    )
+    (property "Datasheet" "~" (at 96.52 110.49 0)
+      (effects (font (size 1.27 1.27)) hide)
+    )
+    (pin "1")
+    (pin "2")
+    (instances
+      (project "relay"
+        (path "/212a0d71-cc7b-49f8-b4ca-a935e5355dca"
+          (reference "R1") (unit 1)
+        )
+      )
+    )
+  )
   (symbol (lib_id "power:GND") (at 66.04 148.59 0) (mirror y) (unit 1)
     (in_bom yes) (on_board yes) (dnp no)
@@
   (symbol (lib_id "Device:C") (at 86.36 118.11 0) (mirror y) (unit 1)
     (in_bom yes) (on_board yes) (dnp no)
-    (property "Reference" "C5" (at 88.9 113.03 0)
+    (property "Reference" "C1" (at 88.9 113.03 0)
       (effects (font (size 1.27 1.27)) (justify left))
     )
@@
       (project "relay"
         (path "/212a0d71-cc7b-49f8-b4ca-a935e5355dca"
-          (reference "C5") (unit 1)
-        )
-      )
+          (reference "C1") (unit 1)
+        )
+      )

Commit message: Increase capacitor value.
Parts:
- C1: value 10u -> 220u; footprint Capacitor_SMD:C_0603_1608Metric -> Capacitor_Tantalum_SMD:CP_EIA-6032-28_Kemet-C
- D2: footprint Diode_SMD:D_SOD-123 -> Diode_SMD:D_MiniMELF
Changed lines of the file:
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@@
       (effects (font (size 1.27 1.27)) (justify right))
     )
-    (property "Footprint" "Diode_SMD:D_SOD-123" (at 77.47 120.65 0)
+    (property "Footprint" "Diode_SMD:D_MiniMELF" (at 77.47 120.65 0)
       (effects (font (size 1.27 1.27)) hide)
     )
@@
   (symbol (lib_id "Device:C") (at 86.36 118.11 0) (mirror y) (unit 1)
     (in_bom yes) (on_board yes) (dnp no)
-    (property "Reference" "C1" (at 88.9 113.03 0)
-      (effects (font (size 1.27 1.27)) (justify left))
-    )
-    (property "Value" "10u" (at 85.09 113.03 0)
-      (effects (font (size 1.27 1.27)) (justify left))
-    )
-    (property "Footprint" "Capacitor_SMD:C_0603_1608Metric" (at 85.3948 121.92 0)
-      (effects (font (size 1.27 1.27)) hide)
-    )
+    (property "Reference" "C1" (at 92.71 116.84 0)
+      (effects (font (size 1.27 1.27)) (justify left))
+    )
+    (property "Value" "220u" (at 95.25 119.38 0)
+      (effects (font (size 1.27 1.27)) (justify left))
+    )
+    (property "Footprint" "Capacitor_Tantalum_SMD:CP_EIA-6032-28_Kemet-C" (at 85.3948 121.92 0)
+      (effects (font (size 1.27 1.27)) hide)
+    )
