File: frontend/pcb/frontend.kicad_sch (KiCad schematic)
At the start: 56 parts, among them J1 Ext, J2 CONN_01X02, J3 Display4020, J4 Debug, J5 RS485, J6 Conn_01x04, J7 Conn_01x02, J8 Conn_01x02, J9 Conn_01x02, K1 G6B-1114C-US5DC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

Commit message: Use Hal9k footprint library.
Parts:
- K1: footprint modules:DIL-relay -> hal9k:DIL-relay
- U4: footprint modules:DSN-MINI-360 -> hal9k:DSN-MINI-360
Changed lines of the file:
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@@
 			)
 		)
-		(property "Footprint" "modules:DIL-relay"
+		(property "Footprint" "hal9k:DIL-relay"
 			(at 236.22 130.81 0)
 			(effects
@@
 			)
 		)
-		(property "Footprint" "modules:DSN-MINI-360"
+		(property "Footprint" "hal9k:DSN-MINI-360"
 			(at 246.38 204.47 0)
 			(effects
