File: frontend/pcb/frontend.kicad_pcb (KiCad board)
At the start: 2 copper layers, 63.6 x 49 mm, 56 parts, among them J1 Ext, J2 CONN_01X02, J3 Display4020, J4 Debug, J5 RS485, J6 Conn_01x04, J7 Conn_01x02, J8 Conn_01x02, J9 Conn_01x02, K1 G6B-1114C-US5DC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

Commit message: Use Hal9k footprint library.
Parts:
- K1: footprint modules:DIL-relay -> hal9k:DIL-relay
- U4: footprint modules:DSN-MINI-360 -> hal9k:DSN-MINI-360

Commit message: Show resistor references on silk screen.
Other:
- board text added: "12"
- board text added: "3.3"
- board text added: "5"
Changed lines of the file:
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@@
 (kicad_pcb
-	(version 20231212)
+	(version 20240108)
 	(generator "pcbnew")
-	(generator_version "7.99")
+	(generator_version "8.99")
 	(general
 		(thickness 1.6)
@@
 		(tags "resistor")
 		(property "Reference" "R10"
-			(at 0 -1.43 180)
+			(at -2.2352 0.1016 -90)
 			(layer "F.SilkS")
-			(hide yes)
 			(effects
 				(font
@@
 		(tags "resistor")
 		(property "Reference" "R16"
-			(at 0 -1.43 0)
+			(at -0.1777 1.6764 0)
 			(layer "F.SilkS")
-			(hide yes)
 			(effects
 				(font
@@
 			(at 0 -1.43 -90)
 			(layer "F.SilkS")
-			(hide yes)
 			(effects
 				(font
@@
 			(at 0 -1.43 90)
 			(layer "F.SilkS")
-			(hide yes)
 			(effects
 				(font
@@
 			(at 2.7685 -0.03 90)
 			(layer "F.SilkS")
-			(hide yes)
 			(effects
 				(font
@@
 		(tags "resistor")
 		(property "Reference" "R1"
-			(at -2.54 -0.508 0)
+			(at -2.794 0 0)
 			(layer "F.SilkS")
-			(hide yes)
 			(effects
 				(font
@@
 			(at 0 1.524 -90)
 			(layer "F.SilkS")
-			(hide yes)
 			(effects
 				(font
@@
 			(at 2.7685 -0.06 90)
 			(layer "F.SilkS")
-			(hide yes)
 			(effects
 				(font
@@
 			(at 2.7685 0.03 90)
 			(layer "F.SilkS")
-			(hide yes)
 			(effects
 				(font
@@
 		(tags "resistor")
 		(property "Reference" "R19"
-			(at 0 -1.43 90)
+			(at 3.2259 -0.0508 90)
 			(layer "F.SilkS")
-			(hide yes)
 			(effects
 				(font
@@
 			(at 0 -1.43 180)
 			(layer "F.SilkS")
-			(hide yes)
 			(effects
 				(font
@@
 		(tags "resistor")
 		(property "Reference" "R13"
-			(at 0 -1.43 0)
+			(at 2.5147 -0.0508 90)
 			(layer "F.SilkS")
-			(hide yes)
 			(effects
 				(font
@@
 		(tags "resistor")
 		(property "Reference" "R14"
-			(at 0 -1.43 0)
+			(at -2.4129 -0.0508 90)
 			(layer "F.SilkS")
-			(hide yes)
 			(effects
 				(font
@@
 		(tags "resistor")
 		(property "Reference" "R20"
-			(at 0 -1.43 0)
+			(at -2.2097 -0.0508 90)
 			(layer "F.SilkS")
-			(hide yes)
 			(effects
 				(font
@@
 			(at -2.8195 0 180)
 			(layer "F.SilkS")
-			(hide yes)
 			(effects
 				(font
@@
 		(tags "resistor")
 		(property "Reference" "R5"
-			(at -2.0575 0.254 180)
+			(at 2.5145 -0.5588 -90)
 			(layer "F.SilkS")
-			(hide yes)
 			(effects
 				(font
@@
 			(at 0 1.524 -90)
 			(layer "F.SilkS")
-			(hide yes)
 			(effects
 				(font
@@
 		(tags "resistor")
 		(property "Reference" "R2"
-			(at 0 -1.43 0)
+			(at 2.54 0.6096 0)
 			(layer "F.SilkS")
-			(hide yes)
 			(effects
 				(font
@@
 			(at 2.7685 0 90)
 			(layer "F.SilkS")
-			(hide yes)
 			(effects
 				(font
@@
 			(at 0 -1.43 -90)
 			(layer "F.SilkS")
-			(hide yes)
 			(effects
 				(font
@@
 		)
 	)
+	(gr_text "5"
+		(at 85.2424 104.6988 0)
+		(layer "F.SilkS")
+		(effects
+			(font
+				(size 1 1)
+				(thickness 0.15)
+			)
+			(justify left bottom)
+		)
+	)
 	(gr_text "GND"
 		(at 55.626 109.982 90)
@@
 		)
 	)
+	(gr_text "3.3"
+		(at 91.8464 104.8004 0)
+		(layer "F.SilkS")
+		(effects
+			(font
+				(size 1 1)
+				(thickness 0.15)
+			)
+			(justify left bottom)
+		)
+	)
 	(gr_text "BOOT"
 		(at 87.376 62.484 0)
@@
 	)
 	(gr_text "LOCK"
-		(at 38.608 82.296 0)
+		(at 46.807321 88.339821 90)
+		(layer "F.SilkS")
+		(effects
+			(font
+				(size 1 1)
+				(thickness 0.15)
+			)
+			(justify left bottom)
+		)
+	)
+	(gr_text "12"
+		(at 44.9445 80.35 0)
 		(layer "F.SilkS")
 		(effects
@@
 	)
 	(gr_text "DOOR"
-		(at 47.244 74.168 90)
+		(at 46.4312 73.914 90)
 		(layer "F.SilkS")
 		(effects
@@
 	)
 	(gr_text "ACS frontend"
-		(at 61.468 75.692 0)
+		(at 60.198 82.3976 22.5)
 		(layer "F.SilkS")
 		(effects
 			(font
-				(size 1 1)
+				(size 1.5 1.5)
 				(thickness 0.15)
 			)
@@
 		(polygon
 			(pts
-				(xy 39.37 62.3824) (xy 100.076 62.1284) (xy 100.2284 108.3564) (xy 39.624 108.6104)
+				(xy 39.591066 102.61646) (xy 39.404058 68.580929) (xy 45.72 68.58) (xy 45.717259 62.30628) (xy 94.4372 61.722)
+				(xy 94.488 68.9356) (xy 100.098438 68.934689) (xy 100.208137 102.209834) (xy 93.8276 102.2604) (xy 93.827712 108.383226)
+				(xy 45.720745 108.584848) (xy 45.72 102.616)
 			)
 		)

Commit message: Remove track fragment
Routing:
- net Net-(J5-Pin_3): track 10.7 -> 10.0 mm
Changed lines of the file:
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@@
-	)
-	(segment
-		(start 72.009 99.695)
-		(end 72.009 98.995)
-		(width 0.2)
-		(layer "F.Cu")
-		(net 21)
 	)
 	(segment
